Commit message: add gazebo sim code

File: assets/go2w_description/urdf/go2w_description.urdf (robot description, URDF)
Before this commit: robot go2w_description, 33 links, 32 joints
Links:
- removed link imu
- removed link radar
- added link imu_link, mass 0
- added link radar_link, mass 0
- added link trunk, mass 6.921; collision box size=0.3762 0.0935 0.114; visual mesh filename=package://go2w_description/meshes/base.dae
- link FL_calf: geometry collision cylinder length=0.12 radius=0.012; visual mesh filename=package://go2w_description/meshes/calf.stl
- link FL_foot: geometry collision mesh filename=package://go2w_description/meshes/left_wheel.dae; visual mesh filename=package://go2w_description/meshes/left_wheel.dae
- link FL_hip: geometry collision cylinder length=0.04 radius=0.046; visual mesh filename=package://go2w_description/meshes/hip.dae
- link FL_thigh: geometry collision box size=0.11 0.0245 0.034; visual mesh filename=package://go2w_description/meshes/thigh.dae
- link FR_calf: geometry collision cylinder length=0.12 radius=0.013; visual mesh filename=package://go2w_description/meshes/calf_mirror.stl
- link FR_foot: geometry collision mesh filename=package://go2w_description/meshes/right_wheel.dae; visual mesh filename=package://go2w_description/meshes/right_wheel.dae
- link FR_hip: geometry collision cylinder length=0.04 radius=0.046; visual mesh filename=package://go2w_description/meshes/hip.dae
- link FR_thigh: geometry collision box size=0.11 0.0245 0.034; visual mesh filename=package://go2w_description/meshes/thigh_mirror.dae
- link RL_calf: geometry collision cylinder length=0.12 radius=0.013; visual mesh filename=package://go2w_description/meshes/calf.stl
- link RL_foot: geometry collision mesh filename=package://go2w_description/meshes/left_wheel.dae; visual mesh filename=package://go2w_description/meshes/left_wheel.dae
- link RL_hip: geometry collision cylinder length=0.04 radius=0.046; visual mesh filename=package://go2w_description/meshes/hip.dae
- link RL_thigh: geometry collision box size=0.11 0.0245 0.034; visual mesh filename=package://go2w_description/meshes/thigh.dae
- link RR_calf: geometry collision cylinder length=0.12 radius=0.013; visual mesh filename=package://go2w_description/meshes/calf_mirror.stl
- link RR_foot: geometry collision mesh filename=package://go2w_description/meshes/right_wheel.dae; visual mesh filename=package://go2w_description/meshes/right_wheel.dae
- link RR_hip: geometry collision cylinder length=0.04 radius=0.046; visual mesh filename=package://go2w_description/meshes/hip.dae
- link RR_thigh: geometry collision box size=0.11 0.0245 0.034; visual mesh filename=package://go2w_description/meshes/thigh_mirror.dae
- link base: mass 6.921 -> None; geometry visual box size=0.001 0.001 0.001
Joints:
- added joint floating_base: type fixed, parent base, child trunk, origin xyz=0 0 0 rpy=0 0 0
- joint FL_foot_joint: limit lower=-999999 upper=999999 effort=23.7 velocity=30.1 -> effort=23.7 velocity=30.1; type revolute -> continuous
- joint FL_hip_joint: parent base -> trunk
- joint FR_foot_joint: limit lower=-999999 upper=999999 effort=23.7 velocity=30.1 -> effort=23.7 velocity=30.1; type revolute -> continuous
- joint FR_hip_joint: parent base -> trunk
- joint Head_upper_joint: parent base -> trunk
- joint RL_foot_joint: limit lower=-999999 upper=999999 effort=23.7 velocity=30.1 -> effort=23.7 velocity=30.1; type revolute -> continuous
- joint RL_hip_joint: parent base -> trunk
- joint RR_foot_joint: limit lower=-999999 upper=999999 effort=23.7 velocity=30.1 -> effort=23.7 velocity=30.1; type revolute -> continuous
- joint RR_hip_joint: parent base -> trunk
- joint imu_joint: child imu -> imu_link; parent base -> trunk
- joint radar_joint: child radar -> radar_link; parent base -> trunk
